File: asterisk60.sch (KiCad schematic (older format))
At the start: 125 parts, among them SW0 MX_LED, SW1 MX_LED, SW10 MX_LED, SW11 MX_LED, SW12 MX_LED, SW13 MX_LED, SW14 MX_LED, SW15 MX_LED, SW16 MX_LED, SW17 MX_LED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

Commit message: revamped pcb and added top and bottom plates
Parts:
- D0, D1, D10, D11, D12, D13, D14, D15, D16, D17, D18, D19, D2, D20, D21, D22, D23, D24, D25, D26, D27, D28, D29, D3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: footprint diode:Diotec_Semiconductor-1N4148-0 -> Diode_THT:D_DO-35_SOD27_P7.62mm_Horizontal
