File: asterisk60platetop.kicad_pcb (KiCad board)
At the start: 2 copper layers, 240 x 106.7 mm, 19 parts

Commit message: logo added
Parts:
- added REF**: origami-logo-sixtyfourth, customlogos:origami-logo-sixtyfourth, F.Cu at (247.7, 121.3)
- added REF**: origami-logo-sixtyfourth, customlogos:origami-logo-sixtyfourth, B.Cu at (228.0, 121.3)
